Commit message: Update URDF files to correspond to actual robot

File: src/diff_drive_robot/description/models/urdf/camera.xacro (robot description, xacro)
@@ -4,5 +4,5 @@
         <parent link="chassis"/>
         <child link="camera_link"/>
-        <origin xyz="0.276 0 0.181" rpy="0 0.18 0"/>
+        <origin xyz="0.237 0 0.045" rpy="0 0 0"/>
     </joint>
     <link name="camera_link">
@@ -10,11 +10,4 @@
             <geometry>
                 <box size="0.010 0.03 0.03"/>
-            </geometry>
-            <material name="black"/>
-        </visual>
-        <visual>
-            <origin xyz="0 0 -0.05"/>
-            <geometry>
-                <cylinder radius="0.002" length="0.1"/>
             </geometry>
             <material name="black"/>

File: src/diff_drive_robot/description/models/urdf/lidar.xacro (robot description, xacro)
@@ -4,5 +4,6 @@
         <parent link="chassis"/>
         <child link="lidar_link"/>
-        <origin xyz="0.122 0 0.212" rpy="0 0 0"/>
+        <!-- Half of chassis forward and chassi height + half of lidar height up -->
+        <origin xyz="0.1175 0 0.11" rpy="0 0 0"/>
     </joint>
     <link name="lidar_link">
@@ -10,11 +11,4 @@
             <geometry>
                 <cylinder radius="0.05" length="0.04"/>
-            </geometry>
-            <material name="black"/>
-        </visual>
-        <visual>
-            <origin xyz="0 0 -0.05"/>
-            <geometry>
-                <cylinder radius="0.01" length="0.1"/>
             </geometry>
             <material name="black"/>

File: src/diff_drive_robot/description/models/urdf/robot.urdf.xacro (robot description, xacro)
@@ -1,4 +1,4 @@
 <?xml version="1.0"?>
-<robot xmlns:xacro="http://www.ros.org/wiki/xacro"  name="robot">
+<robot xmlns:xacro="http://www.ros.org/wiki/xacro"  name="diff_drive">
     <xacro:include filename="robot_core.xacro" />
     <xacro:include filename="ros2_control.xacro" />

File: src/diff_drive_robot/description/models/urdf/robot_core.xacro (robot description, xacro)
@@ -1,4 +1,4 @@
 <?xml version="1.0"?>
-<robot xmlns:xacro="http://www.ros.org/wiki/xacro" name="diff_drive">
+<robot xmlns:xacro="http://www.ros.org/wiki/xacro">
     <xacro:include filename="inertial_macros.xacro"/>
     <xacro:property name="chassis_length" value="0.235"/>
@@ -6,10 +6,10 @@
     <xacro:property name="chassis_height" value="0.09"/>
     <xacro:property name="chassis_mass" value="1.0"/>
-    <xacro:property name="wheel_radius" value="0.033"/>
-    <xacro:property name="wheel_thickness" value="0.026"/>
+    <xacro:property name="wheel_radius" value="0.0325"/>
+    <xacro:property name="wheel_thickness" value="0.03"/>
     <xacro:property name="wheel_mass" value="0.05"/>
-    <xacro:property name="wheel_offset_x" value="0.226"/>
-    <xacro:property name="wheel_offset_y" value="0.1485"/>
-    <xacro:property name="wheel_offset_z" value="0.01"/>
+    <xacro:property name="wheel_offset_x" value="0.05"/>
+    <xacro:property name="wheel_offset_y" value="0.14"/>
+    <xacro:property name="wheel_offset_z" value="0.0205"/>
     <xacro:property name="caster_wheel_radius" value="0.01"/>
     <xacro:property name="caster_wheel_mass" value="0.01"/>
@@ -34,14 +34,22 @@
     <!-- Seems to needed to not get warnings in Rviz -->
     <link name="base_link">
+        <origin xyz="2 0 0"/>
+    </link>
+     <joint name="base_footprint_joint" type="fixed">
+        <parent link="base_link"/>
+        <child link="base_footprint"/>
+        <origin xyz="0 0 0" rpy="0 0 0"/>
+    </joint>
+    <link name="base_footprint">
     </link>
     <!-- CHASSIS LINK -->
-    <joint name="chassis_joint" type="fixed">
+     <joint name="chassis_joint" type="fixed">
         <parent link="base_link"/>
         <child link="chassis"/>
-        <origin xyz="0 0 0"/>
+        <origin xyz="${-wheel_offset_x} 0 ${-wheel_offset_z}"/>
     </joint>
     <link name="chassis">
         <visual>
-            <origin xyz="0 0 0"/>
+             <origin xyz="${chassis_length/2} 0 ${chassis_height/2}"/>
             <geometry>
                 <box size="0.235 0.235 0.09"/>
@@ -50,9 +58,12 @@
         </visual>
         <collision>
-            <origin xyz="0 0 0"/>
+             <origin xyz="${chassis_length/2} 0 ${chassis_height/2}"/>
             <geometry>
                 <box size="0.235 0.235 0.09"/>
             </geometry>
         </collision>
+         <xacro:inertial_box mass="0.5" x="${chassis_length}" y="${chassis_width}" z="${chassis_height}">
+            <origin xyz="${chassis_length/2} 0 ${chassis_height/2}" rpy="0 0 0"/>
+        </xacro:inertial_box>
     </link>
     <!-- LEFT WHEEL LINK -->
@@ -75,4 +86,7 @@
             </geometry>
         </collision>
+        <xacro:inertial_cylinder mass="${wheel_mass}" length="${wheel_thickness}" radius="${wheel_radius}">
+            <origin xyz="0 0 0" rpy="0 0 0"/>
+        </xacro:inertial_cylinder>
     </link>
     <!-- RIGHT WHEEL LINK -->
@@ -80,5 +94,5 @@
         <parent link="base_link"/>
         <child link="right_wheel"/>
-        <origin xyz="0 0 0" rpy="0 0 0" />
+        <origin xyz="0 ${-wheel_offset_y} 0" rpy="${pi/2} 0 0" />
         <axis xyz="0 0 -1"/>
     </joint>
@@ -95,4 +109,7 @@
             </geometry>
         </collision>
+        <xacro:inertial_cylinder mass="${wheel_mass}" length="${wheel_thickness}" radius="${wheel_radius}">
+            <origin xyz="0 0 0" rpy="0 0 0"/>
+        </xacro:inertial_cylinder>
     </link>
     <!-- CASTER WHEEL LINK -->
@@ -100,5 +117,5 @@
         <parent link="chassis"/>
         <child link="caster_wheel"/>
-        <origin xyz="0 0 0"/>
+        <origin xyz="${caster_wheel_offset_x + (chassis_length/2)} 0 ${caster_wheel_offset_z}"/>
     </joint>
     <link name="caster_wheel">
@@ -114,4 +131,7 @@
             </geometry>
         </collision>
+        <xacro:inertial_sphere mass="${caster_wheel_mass}" radius="${caster_wheel_radius}">
+            <origin xyz="0 0 0" rpy="0 0 0"/>
+        </xacro:inertial_sphere>
     </link>
     <gazebo reference="caster_wheel">
