Commit message: Fix lidar for gazebo

File: src/diff_drive_robot/description/models/urdf/lidar.xacro (robot description, xacro)
@@ -23,3 +23,34 @@
         </xacro:inertial_cylinder>
     </link>
+     <gazebo reference="lidar_link">
+        <material>Gazebo/Black</material>
+<sensor name='gpu_lidar' type='gpu_lidar'>
+          <pose>0 0 0 0 0 0</pose>
+          <topic>scan</topic>
+          <ignition_frame_id>lidar_link</ignition_frame_id>
+          <update_rate>10</update_rate>
+          <lidar>
+            <scan>
+              <horizontal>
+                <samples>640</samples>
+                <resolution>1</resolution>
+                <min_angle>-3.14</min_angle>
+                <max_angle>3.14</max_angle>
+              </horizontal>
+              <vertical>
+                <samples>1</samples>
+                <resolution>1</resolution>
+                <min_angle>0.0</min_angle>
+                <max_angle>0.0</max_angle>
+              </vertical>
+            </scan>
+            <range>
+              <min>0.08</min>
+              <max>10.0</max>
+              <resolution>0.01</resolution>
+            </range>
+          </lidar>
+          <visualize>true</visualize>
+        </sensor>
+         </gazebo>
 </robot>
