Commit message: Remove base footprint, not sure what it is for

File: src/diff_drive_robot/description/models/urdf/robot_core.xacro (robot description, xacro)
@@ -35,11 +35,4 @@
     <link name="base_link">
         <origin xyz="2 0 0"/>
-    </link>
-     <joint name="base_footprint_joint" type="fixed">
-        <parent link="base_link"/>
-        <child link="base_footprint"/>
-        <origin xyz="0 0 0" rpy="0 0 0"/>
-    </joint>
-    <link name="base_footprint">
     </link>
     <!-- CHASSIS LINK -->

Commit message: add base footprint for map

File: src/diff_drive_robot/description/models/urdf/robot_core.xacro (robot description, xacro)
@@ -32,7 +32,13 @@
     </material>
     <!-- BASE LINK -->
-    <!-- Seems to needed to not get warnings in Rviz -->
     <link name="base_link">
         <origin xyz="2 0 0"/>
+    </link>
+    <joint name="base_footprint_joint" type="fixed">
+        <parent link="base_link"/>
+        <child link="base_footprint"/>
+        <origin xyz="0 0 0" rpy="0 0 0"/>
+    </joint>
+    <link name="base_footprint">
     </link>
     <!-- CHASSIS LINK -->
