Commit message: Prepare to launch code on robot

File: src/diff_drive_robot/description/models/urdf/ros2_control.xacro (robot description, xacro)
@@ -1,64 +1,34 @@
 <?xml version="1.0"?>
 <robot xmlns:xacro="http://www.ros.org/wiki/xacro">
-    <!-- <xacro:unless value="$(arg sim_mode)"> -->
-        <!-- <ros2_control name="RealRobot" type="system">
-            <hardware>
-                <plugin>diffdrive_arduino/DiffDriveArduino</plugin>
-                <param name="left_wheel_name">left_wheel_joint</param>
-                <param name="right_wheel_name">right_wheel_joint</param>
-                <param name="loop_rate">30</param>
-                <param name="device">/dev/ttyUSB0</param>
-                <param name="baud_rate">57600</param>
-                <param name="timeout">1000</param>
-                <param name="enc_counts_per_rev">3436</param>
-            </hardware>
-            <joint name="left_wheel_joint">
-                <command_interface name="velocity">
-                    <param name="min">-10</param>
-                    <param name="max">10</param>
-                </command_interface>
-                <state_interface name="velocity"/>
-                <state_interface name="position"/>
-            </joint>
-            <joint name="right_wheel_joint">
-                <command_interface name="velocity">
-                    <param name="min">-10</param>
-                    <param name="max">10</param>
-                </command_interface>
-                <state_interface name="velocity"/>
-                <state_interface name="position"/>
-            </joint>
-        </ros2_control> -->
-    <!-- </xacro:unless> -->
-    <!-- <xacro:if value="$(arg sim_mode)">
-        <ros2_control name="GazeboSystem" type="system">
-            <hardware>
-                <plugin>gazebo_ros2_control/GazeboSystem</plugin>
-            </hardware>
-            <joint name="left_wheel_joint">
-                <command_interface name="velocity">
-                    <param name="min">-10</param>
-                    <param name="max">10</param>
-                </command_interface>
-                <state_interface name="velocity"/>
-                <state_interface name="position"/>
-            </joint>
-            <joint name="right_wheel_joint">
-                <command_interface name="velocity">
-                    <param name="min">-10</param>
-                    <param name="max">10</param>
-                </command_interface>
-                <state_interface name="velocity"/>
-                <state_interface name="position"/>
-            </joint>
-        </ros2_control>
-    </xacro:if> -->
-    <!-- <gazebo>
-        <plugin name="gazebo_ros2_control" filename="libgazebo_ros2_control.so">
-            <parameters>$(find articubot_one)/config/my_controllers.yaml</parameters> -->
-            <!-- <parameters>$(find articubot_one)/config/gaz_ros2_ctl_use_sim.yaml</parameters> -->
-        <!-- </plugin>
-    </gazebo> -->
-    <ros2_control name="IgnitionSystem" type="system">
+    <ros2_control name="RealRobot" type="system">
+        <hardware>
+            <plugin>diffdrive_arduino/DiffDriveArduino</plugin>
+            <param name="left_wheel_name">left_wheel_joint</param>
+            <param name="right_wheel_name">right_wheel_joint</param>
+            <param name="loop_rate">30</param>
+            <param name="device">/dev/ttyUSB0</param>
+            <param name="baud_rate">57600</param>
+            <param name="timeout">1000</param>
+            <param name="enc_counts_per_rev">2400</param>
+        </hardware>
+        <joint name="left_wheel_joint">
+            <command_interface name="velocity">
+                <param name="min">-10</param>
+                <param name="max">10</param>
+            </command_interface>
+            <state_interface name="velocity"/>
+            <state_interface name="position"/>
+        </joint>
+        <joint name="right_wheel_joint">
+            <command_interface name="velocity">
+                <param name="min">-10</param>
+                <param name="max">10</param>
+            </command_interface>
+            <state_interface name="velocity"/>
+            <state_interface name="position"/>
+        </joint>
+    </ros2_control>
+    <!-- Needed for gazebo control -->
+    <!-- <ros2_control name="IgnitionSystem" type="system">
         <hardware>
           <plugin>ign_ros2_control/IgnitionSystem</plugin>
@@ -80,10 +50,4 @@
           <state_interface name="velocity"/>
         </joint>
-      </ros2_control>
-<!--
-      <gazebo>
-        <plugin filename="ign_ros2_control-system" name="ign_ros2_control::IgnitionROS2ControlPlugin">
-              <parameters>/home/mikaeltrana/Documents/robot/my_bot/install/bringup/share/bringup/config/my_controller.yaml</parameters>
-        </plugin>
-    </gazebo> -->
+      </ros2_control> -->
 </robot>

Commit message: Use my own hardware for control

File: src/diff_drive_robot/description/models/urdf/ros2_control.xacro (robot description, xacro)
@@ -2,7 +2,7 @@
 <robot xmlns:xacro="http://www.ros.org/wiki/xacro">
     <xacro:unless value="$(arg sim_mode)">
-        <ros2_control name="RealRobot" type="system">
+        <ros2_control name="DiffBot" type="system">
             <hardware>
-                <plugin>diffdrive_arduino/DiffDriveArduino</plugin>
+                <plugin>diffdrive_arduino/DiffBotArduinoHardware</plugin>
                 <param name="left_wheel_name">left_wheel_joint</param>
                 <param name="right_wheel_name">right_wheel_joint</param>
@@ -10,8 +10,23 @@
                 <param name="device">/dev/serial/by-id/usb-FTDI_FT232R_USB_UART_B0015R0O-if00-port0</param>
                 <param name="baud_rate">57600</param>
-                <param name="timeout">1000</param>
-                <param name="enc_counts_per_rev">2400</param>
+                <param name="timeout_ms">1000</param>
+                <param name="left_wheel_enc_counts_per_rev">3000</param>
+                <param name="right_wheel_enc_counts_per_rev">2000</param>
+                <param name="pid_p">20</param>
+                <param name="pid_d">12</param>
+                <param name="pid_i">0</param>
+                <param name="pid_o">50</param>
             </hardware>
-            <joint name="left_wheel_joint">
+<joint name="left_wheel_joint">
+        <command_interface name="velocity"/>
+        <state_interface name="position"/>
+        <state_interface name="velocity"/>
+      </joint>
+      <joint name="right_wheel_joint">
+        <command_interface name="velocity"/>
+        <state_interface name="position"/>
+        <state_interface name="velocity"/>
+      </joint>
+            <!-- <joint name="left_wheel_joint">
                 <command_interface name="velocity">
                     <param name="min">-10</param>
@@ -28,5 +43,5 @@
                 <state_interface name="velocity"/>
                 <state_interface name="position"/>
-            </joint>
+            </joint> -->
         </ros2_control>
     </xacro:unless>
